Commit message: Imported upstream version '1.1.0' of 'upstream'

File: vrx_gazebo/worlds/example_course.world.xacro (robot description, xacro)
@@ -7,9 +7,9 @@
     <include>
       <uri>model://robotx_navigation_challenge</uri>
-      <pose>15 0 2 0 0 0</pose>
+      <pose>58 68 2 0 0 0.4</pose>
     </include>
     <include>
       <uri>model://robotx_light_buoy</uri>
-      <pose>60 0 0.25 0 0 0</pose>
+      <pose>110 28 0.25 0 0 0</pose>
     </include>
     <include>
@@ -20,11 +20,21 @@
     <include>
       <uri>model://dock_2016</uri>
-      <pose>80 -8.75 0 0 0 0</pose>
+      <pose>75 22 0 0 0 -2.78</pose>
     </include>
     <!-- The 2018 dock with the two placards -->
     <include>
       <uri>model://dock_2018</uri>
-      <pose>120 -2.75 0 0 0 0</pose>
+      <pose>-2 -18 0 0 0 0.2</pose>
     </include>
+    <xacro:include filename="$(find vrx_gazebo)/worlds/xacros/usv_wind_plugin.xacro"/>
+    <xacro:usv_wind_gazebo>
+      <wind_objs>
+        <wind_obj>
+          <name>wamv</name>
+          <link_name>base_link</link_name>
+          <coeff_vector>.5 .5 .33</coeff_vector>
+        </wind_obj>
+      </wind_objs>
+    </xacro:usv_wind_gazebo>
   </world>
 </sdf>

File: vrx_gazebo/worlds/navigation_task.world.xacro (robot description, xacro)
@@ -5,121 +5,19 @@
     <xacro:include filename="$(find vrx_gazebo)/worlds/sandisland.xacro" />
     <xacro:sandisland />
-    <!-- Starboard_border -->
+    <!--wind for the wamv-->
+    <xacro:include filename="$(find vrx_gazebo)/worlds/xacros/usv_wind_plugin.xacro"/>
+    <xacro:usv_wind_gazebo direction = "270" ros_update_rate="10">
+      <wind_objs>
+        <wind_obj>
+          <name>wamv</name>
+          <link_name>base_link</link_name>
+          <coeff_vector>.5 .5 .33</coeff_vector>
+        </wind_obj>
+      </wind_objs>
+    </xacro:usv_wind_gazebo>
+    <!-- The VRX navigation course -->
     <include>
-        <name>red_bound_0</name>
-        <pose>-29.8874 7.80274 0 0 -0 0</pose>
-        <uri>model://surmark950410</uri>
-      </include>
-    <include>
-      <name>red_bound_1</name>
-      <pose>-51.4227 1.0515 0 0 -0 0</pose>
-      <uri>model://surmark950410</uri>
-    </include>
-    <include>
-      <name>red_bound_2</name>
-      <pose>-64.574 -13.7242 0 0 -0 0</pose>
-      <uri>model://surmark950410</uri>
-    </include>
-    <include>
-      <name>red_bound_3</name>
-      <pose>-70.5798 -30.9289 0 0 -0 0</pose>
-      <uri>model://surmark950410</uri>
-    </include>
-    <include>
-      <name>red_bound_4</name>
-      <pose>-73.2084 -44.9953 0 0 -0 0</pose>
-      <uri>model://surmark950410</uri>
-    </include>
-    <include>
-      <name>red_bound_5</name>
-      <pose>-87.3051 -43.4804 0 0 -0 0</pose>
-      <uri>model://surmark950410</uri>
-    </include>
-    <include>
-      <name>red_bound_6</name>
-      <pose>-90.539 -28.0283 0 0 -0 0</pose>
-      <uri>model://surmark950410</uri>
-    </include>
-    <!-- Port_border -->
-    <include>
-      <name>green_bound_0</name>
-      <pose>-32.2914 -10.0761 -0.2 0 -0 0</pose>
-      <uri>model://surmark950400</uri>
-    </include>
-    <include>
-      <name>green_bound_1</name>
-      <pose>-47.3915 -11.2422 -0.2 0 -0 0</pose>
-      <uri>model://surmark950400</uri>
-    </include>
-    <include>
-      <name>green_bound_2</name>
-      <pose>-50.4509 -25.1164 -0.2 0 -0 0</pose>
-      <uri>model://surmark950400</uri>
-    </include>
-    <include>
-      <name>green_bound_3</name>
-      <pose>-58.7734 -39.351 -0.2 0 -0 0</pose>
-      <uri>model://surmark950400</uri>
-    </include>
-    <include>
-      <name>green_bound_4</name>
-      <pose>-70.9557 -57.7238 -0.2 0 -0 0</pose>
-      <uri>model://surmark950400</uri>
-    </include>
-    <include>
-      <name>green_bound_5</name>
-      <pose>-95.8278 -54.0979 -0.2 0 -0 0</pose>
-      <uri>model://surmark950400</uri>
-    </include>
-    <include>
-      <name>green_bound_6</name>
-      <pose>-107.643 -29.1729 -0.2 0 -0 0</pose>
-      <uri>model://surmark950400</uri>
-    </include>
-    <!-- Obstacles -->
-    <include>
-      <name>obstacle_1</name>
-      <pose>-57.283 -28.3719 -0.2 0 -0 0</pose>
-      <uri>model://polyform_a5</uri>
-    </include>
-    <include>
-      <name>obstacle_2</name>
-      <pose>-68.6471 -41.2087 -0.2 0 -0 0</pose>
-      <uri>model://polyform_a5</uri>
-    </include>
-    <include>
-      <name>obstacle_3</name>
-      <pose>-80.2333 -48.5559 -0.2 0 -0 0</pose>
-      <uri>model://polyform_a5</uri>
-    </include>
-    <include>
-      <name>obstacle_4</name>
-      <pose>-78.842 -55.2626 -0.2 0 -0 0</pose>
-      <uri>model://polyform_a5</uri>
-    </include>
-    <include>
-      <name>obstacle_5</name>
-      <pose>-84.9105 -53.4974 -0.2 0 -0 0</pose>
-      <uri>model://polyform_a5</uri>
-    </include>
-    <include>
-      <name>obstacle_6</name>
-      <pose>-98.5759 -42.8883 -0.2 0 -0 0</pose>
-      <uri>model://polyform_a5</uri>
-    </include>
-    <include>
-      <name>obstacle_7</name>
-      <pose>-95.2334 -39.1624 -0.2 0 -0 0</pose>
-      <uri>model://polyform_a5</uri>
-    </include>
-    <include>
-      <name>obstacle_8</name>
-      <pose>-100.506 -33.524 -0.2 0 -0 0</pose>
-      <uri>model://polyform_a5</uri>
-    </include>
-    <include>
-      <name>obstacle_9</name>
-      <pose>-56.0734 -9.21053 -0.2 0 -0 0</pose>
-      <uri>model://polyform_a7</uri>
+      <uri>model://navigation_course</uri>
+      <pose>130 100 0 0 0 0</pose>
     </include>
     <!-- The scoring plugin -->
@@ -131,4 +29,5 @@
       <ready_state_duration>10</ready_state_duration>
       <running_state_duration>300</running_state_duration>
+      <collision_buffer>10</collision_buffer>
       <release_joints>
         <joint>
@@ -139,4 +38,6 @@
         </joint>
       </release_joints>
+      <course_name>vrx_navigation_course</course_name>
+      <obstacle_penalty>10.0</obstacle_penalty>
       <gates>
         <gate>

File: vrx_gazebo/worlds/perception_task.world.xacro (robot description, xacro)
@@ -5,53 +5,56 @@
     <xacro:include filename="$(find vrx_gazebo)/worlds/sandisland.xacro" />
     <xacro:sandisland />
-	<!-- Include all the objects we plan to use for perception.
-		 Stash them out of the field of view for now -->
-	<include>
-	  <name>red_0</name>
-	  <pose>-20 0 1 0 0 0</pose>
-	  <uri>model://surmark950410</uri>
-	</include>
-	<include>
-	  <name>green_0</name>
-	  <pose>-22 0 1 0 0 0</pose>
-	  <uri>model://surmark950400</uri>
-	</include>
-	<include>
-	  <name>black_0</name>
-	  <pose>-24 0 1 0 0 0</pose>
-	  <uri>model://black_totem</uri>
-	</include>
-	<plugin filename="libperception_scoring_plugin.so"
-			name="perception_scoring_plugin">
-	  <!-- Parameters for ScoringPlugin base class -->
-	  <vehicle>wamv</vehicle>
+    <!-- Include all the objects we plan to use for perception.
+       Stash them out of the field of view for now -->
+    <include>
+      <name>red_0</name>
+      <pose>-200 100 1 0 0 0</pose>
+      <uri>model://surmark950410</uri>
+    </include>
+    <include>
+      <name>green_0</name>
+      <pose>-200 102 1 0 0 0</pose>
+      <uri>model://surmark950400</uri>
+    </include>
+    <include>
+      <name>black_0</name>
+      <pose>-200 104 1 0 0 0</pose>
+      <uri>model://black_totem</uri>
+    </include>
+    <plugin filename="libperception_scoring_plugin.so"
+            name="perception_scoring_plugin">
+      <!-- Parameters for ScoringPlugin base class -->
+      <vehicle>wamv</vehicle>
       <task_name>perception</task_name>
-      <initial_state_duration>1</initial_state_duration>
-      <ready_state_duration>1</ready_state_duration>
+      <initial_state_duration>10.0</initial_state_duration>
+      <ready_state_duration>10.0</ready_state_duration>
       <running_state_duration>300</running_state_duration>
-	  <!-- Parameters for PopulationPlugin -->
-	  <loop_forever>false</loop_forever>
-	  <frame>wamv</frame>
-	  <object_sequence>
-		<object>
-		  <time>10.0</time>
-		  <type>red</type>
-		  <name>red_mark</name>
-	  	  <pose>6 0 1 0 0 0</pose>
-		</object>
-		<object>
-		  <time>10.0</time>
-		  <type>green</type>
-		  <name>green_mark</name>
-		  <pose>8 2 1 0 0 0</pose>
-		</object>
-		<object>
-		  <time>10.0</time>
-		  <type>black</type>
-		  <name>black_totem</name>
-		  <pose>10 -2 1 0 0 0</pose>
-		</object>
-	  </object_sequence>
-	</plugin>
+      <!-- Parameters for PopulationPlugin -->
+      <loop_forever>false</loop_forever>
+      <frame>wamv</frame>
+      <!-- Pose of each object is expressed relative to the body frame
+           of the object named in the frame field - i.e., relative to
+           the wam-v-->
+      <object_sequence>
+        <object>
+          <time>5.0</time>
+          <type>red</type>
+          <name>red_mark</name>
+            <pose>8 0 1 0 0 0</pose>
+        </object>
+        <object>
+          <time>10.0</time>
+          <type>green</type>
+          <name>green_mark</name>
+          <pose>8 2 1 0 0 0</pose>
+        </object>
+        <object>
+          <time>15.0</time>
+          <type>black</type>
+          <name>black_totem</name>
+          <pose>8 -2 1 0 0 0</pose>
+        </object>
+      </object_sequence>
+    </plugin>
   </world>
 </sdf>

File: vrx_gazebo/worlds/sandisland.world.xacro (robot description, xacro)
@@ -5,4 +5,15 @@
     <xacro:include filename="$(find vrx_gazebo)/worlds/sandisland.xacro" />
     <xacro:sandisland />
+    <!--wind for the wamv-->
+    <xacro:include filename="$(find vrx_gazebo)/worlds/xacros/usv_wind_plugin.xacro"/>
+    <xacro:usv_wind_gazebo mean_vel="1">
+      <wind_objs>
+        <wind_obj>
+          <name>wamv</name>
+          <link_name>base_link</link_name>
+          <coeff_vector>0.5 0.5 0.33</coeff_vector>
+        </wind_obj>
+      </wind_objs>
+    </xacro:usv_wind_gazebo>
   </world>
 </sdf>

File: vrx_gazebo/worlds/sandisland.xacro (robot description, xacro)
@@ -9,4 +9,6 @@
         </clouds>
       </sky>
+      <grid>0</grid>
+      <origin_visual>0</origin_visual>
     </scene>
     <!-- Estimated latitude/longitude of sandisland from satellite imagery -->
@@ -26,7 +28,8 @@
     <gui fullscreen='0'>
       <camera name='user_camera'>
-        <pose frame=''>17.5798 4.82061 4.05674 0 0.216 -2.876</pose>
+        <pose frame=''>175.544 123.61 4.70958 0 0.168 -2.40718</pose>
         <view_controller>orbit</view_controller>
       </camera>
+      <!--<plugin name="GUITaskWidget" filename="libgui_task_widget.so"/>-->
     </gui>
     <include>
@@ -40,5 +43,67 @@
     <include>
       <pose> 0 0 0 0 0 0 </pose>
-      <uri>model://ocean</uri>
+      <uri>model://ocean_waves</uri>
+    </include>
+    <!-- The posts for securing the WAM-V -->
+    <include>
+      <name>post_0</name>
+      <pose>169.22 112.06 0.47 0.046 -0.157 0</pose>
+      <uri>model://post</uri>
+    </include>
+    <include>
+      <name>post_1</name>
+      <pose>173.558 100.809 0.42 0.046 -0.157 0</pose>
+      <uri>model://post</uri>
+    </include>
+    <include>
+      <name>post_2</name>
+      <pose>177.64 90.86 0.3 0.046 -0.157 0</pose>
+      <uri>model://post</uri>
+    </include>
+    <!-- Antenna for communication with the WAM-V -->
+    <include>
+      <pose>175.69 114.29 1.37 0 0 2.00</pose>
+      <uri>model://antenna</uri>
+    </include>
+    <!-- ground station tents -->
+    <include>
+      <name>ground_station_0</name>
+      <pose>177.61 117.20 1.55 0 0 3.54</pose>
+      <uri>model://ground_station</uri>
+    </include>
+    <include>
+      <name>ground_station_1</name>
+      <pose>179.16 113.73 1.55 0 0 3.54</pose>
+      <uri>model://ground_station</uri>
+    </include>
+    <include>
+      <name>ground_station_2</name>
+      <pose>180.61 110.31 1.55 0 0 3.54</pose>
+      <uri>model://ground_station</uri>
+    </include>
+    <include>
+      <name>ground_station_3</name>
+      <pose>182.05 106.83 1.55 0 0 3.54</pose>
+      <uri>model://ground_station</uri>
+    </include>
+    <include>
+      <name>ground_station_4</name>
+      <pose>183.71 103.14 1.55 0 0 3.54</pose>
+      <uri>model://ground_station</uri>
+    </include>
+    <include>
+      <name>ground_station_5</name>
+      <pose>185.28 99.51 1.55 0 0 3.54</pose>
+      <uri>model://ground_station</uri>
+    </include>
+    <include>
+      <name>ground_station_6</name>
+      <pose>186.80 96.02 1.55 0 0 3.54</pose>
+      <uri>model://ground_station</uri>
+    </include>
+    <include>
+      <name>ground_station_7</name>
+      <pose>188.17 92.45 1.55 0 0 3.54</pose>
+      <uri>model://ground_station</uri>
     </include>
   </xacro:macro>

File: vrx_gazebo/worlds/stationkeeping_task.world.xacro (robot description, xacro)
@@ -10,5 +10,5 @@
       <task_name>stationkeeping</task_name>
       <!-- Goal as Latitude, Longitude, Yaw -->
-      <goal_pose>21.31 -157.89 0.0 </goal_pose>
+      <goal_pose>21.31091 -157.88868 0.0 </goal_pose>
       <initial_state_duration>10</initial_state_duration>
       <ready_state_duration>10</ready_state_duration>

File: wamv_description/urdf/wamv_base.urdf.xacro (robot description, xacro)
@@ -81,6 +81,12 @@
     </collision>
   </xacro:macro>
+  <link name="base_link">
+  </link>
+  <joint name="dummy_joint" type = "fixed">
+    <parent link="base_link"/>
+    <child link="dummy_link"/>
+  </joint>
   <!-- Basic model of the 16' WAM-V USV -->
-  <link name="base_link">
+  <link name="dummy_link">
     <visual>
       <geometry>

File: wamv_gazebo/urdf/dynamics/wamv_gazebo_dynamics_plugin.xacro (robot description, xacro)
@@ -25,20 +25,11 @@
         <!-- General dimensions -->
         <!--<boatArea>2.2</boatArea>-->
-		<hullRadius>0.213</hullRadius>
+        <hullRadius>0.213</hullRadius>
         <boatWidth>2.4</boatWidth>
         <boatLength>4.9</boatLength>
-		<!-- Length discretization, AKA, "N" -->
-		<length_n>2</length_n>
-        <!-- Waves x3 -->
-        <wave_n>3</wave_n>
-        <wave_amp0>0.06</wave_amp0>
-        <wave_period0>12.6</wave_period0>
-        <wave_direction0>-1 0</wave_direction0>
-        <wave_amp1>0.04</wave_amp1>
-        <wave_period1>3.7</wave_period1>
-        <wave_direction1>-0.7 0.7</wave_direction1>
-        <wave_amp2>0.03</wave_amp2>
-        <wave_period2>6.3</wave_period2>
-        <wave_direction2>0.7 0.7</wave_direction2>
+        <!-- Length discretization, AKA, "N" -->
+        <length_n>2</length_n>
+        <!-- Wave model -->
+        <wave_model>ocean_waves</wave_model>
       </plugin>
     </gazebo>

File: wamv_gazebo/urdf/macros.xacro (robot description, xacro)
@@ -5,5 +5,4 @@
   <!-- Include dynamics macros -->
   <xacro:include filename="$(find wamv_gazebo)/urdf/dynamics/wamv_gazebo_dynamics_plugin.xacro" />
-  <xacro:include filename="$(find wamv_gazebo)/urdf/dynamics/wamv_gazebo_wind_plugin.xacro" />
   <!-- Include sensor macros -->
   <xacro:include filename="$(find wamv_gazebo)/urdf/sensors/wamv_camera.xacro" />
@@ -12,4 +11,5 @@
   <xacro:include filename="$(find wamv_gazebo)/urdf/sensors/wamv_planar_lidar.xacro" />
   <xacro:include filename="$(find wamv_gazebo)/urdf/sensors/wamv_3d_lidar.xacro" />
+  <xacro:include filename="$(find wamv_gazebo)/urdf/sensors/lidar.xacro" />
   <xacro:include filename="$(find wamv_gazebo)/urdf/sensors/wamv_p3d.xacro" />
 </robot>

File: wamv_gazebo/urdf/sensors/wamv_3d_lidar.xacro (robot description, xacro)
@@ -2,8 +2,16 @@
 <robot xmlns:xacro="http://ros.org/wiki/xacro">
   <!-- Macro to insert a 3D scanning LIDAR with ROS integration
+    name: Prefix used for naming.
+    x: X position of the laser (from the base_link).
+    y: Y position of the laser (from the base_link).
+    z: Z position of the laser (from the base_link).
+    R: Roll orientation of the laser (from the laser's origin).
+    P: Pitch orientation of the laser (from the laser's origin).
+    Y: Yaw orientation of the laser (from the laser's origin).
+    post_Y: Yaw orientation of the post (from the post's origin).
     update_rate: frequency to publish output, hz
     vertical_lasers: number of vertical lasers which spin about Z to generate output
     samples: number of samples during spin, higher is more dense but slows down simulation
-    resolution: proportion of samples to actually simulate, rest are interprolated. Ex: 0.1 means 9/10 samples are interprolated
+    resolution: This number is multiplied by samples to determine the number of range data points returned.
     min_angle: the horizontal angle that the scan begins at
     max_angle: the angle that the scan ends at
@@ -13,22 +21,116 @@
     noise_stddev: Standard deviation of gaussian noise applied to output pointcloud
   -->
-  <xacro:macro name="wamv_3d_lidar" params="name x:=0.7 y:=0 z:=1.45 R:=0 P:=0 Y:=0
-                                            update_rate:=10 vertical_lasers:=16 samples:=1800 resolution:=0.1
+  <xacro:macro name="wamv_3d_lidar" params="name
+                                            x:=0.7 y:=0 z:=1.8
+                                            R:=0 P:=0 Y:=0
+                                            post_Y:=0
+                                            update_rate:=10 vertical_lasers:=16 samples:=1875 resolution:=0.1
                                             min_angle:=${-pi} max_angle:=${pi}
                                             min_vertical_angle:=${-pi/12} max_vertical_angle:=${pi/12}
-                                            max_range:=100 noise_stddev:=0.01">
+                                            max_range:=130 noise_stddev:=0.01">
+    <!-- Define length variables for link positioning -->
+    <xacro:property name="platform_z" value="1.2965"/>
+    <xacro:property name="post_to_post_arm_x" value="0.03"/>
+    <xacro:property name="post_arm_to_lidar_x" value="0.04"/>
+    <xacro:property name="post_arm_to_lidar_z" value="0.05"/>
+    <!-- 3d lidar sensor -->
     <link name="${name}_link">
-      <visual name="${name}_visual">>
+      <visual name="${name}_visual">
+        <origin xyz="0 0 -0.035" rpy="0 0 0"/>
         <geometry>
-          <cylinder radius="0.025" length="0.1" />
+          <mesh filename="package://vrx_gazebo/models/3d_lidar/mesh/3d_lidar.dae"/>
         </geometry>
-        <material name="${name}_visual_material">
-          <color rgba="0.5 1.0 0.5 1.0" />
+      </visual>
+      <collision name="${name}_collision">
+        <geometry>
+          <cylinder radius="0.055" length="0.075"/>
+        </geometry>
+      </collision>
+      <inertial>
+        <mass value="1"/>
+        <inertia
+          ixx="0.00109375"
+          iyy="0.00109375"
+          izz="0.00125"
+          ixy="0"
+          ixz="0"
+          iyz="0"/>
+      </inertial>
+    </link>
+    <!-- Define post length and mass based on desired z position of sensor -->
+    <xacro:property name="post_length" value="${z-platform_z-post_arm_to_lidar_z}"/>
+    <xacro:property name="post_mass_per_meter" value="0.9"/>
+    <xacro:property name="post_mass" value="${post_mass_per_meter * post_length}"/>
+    <xacro:property name="post_radius" value="0.0076"/>
+    <!-- Sensor post -->
+    <link name="${name}_post_link">
+      <visual>
+        <geometry>
+          <cylinder radius="${post_radius}" length="${post_length}"/>
+        </geometry>
+        <material name="${name}_post_material">
+          <color rgba="0.0 0.0 0.0 1.0"/>
         </material>
       </visual>
+      <collision name="${name}_post_collision">
+        <geometry>
+          <cylinder radius="${post_radius}" length="${post_length}"/>
+        </geometry>
+      </collision>
+      <inertial>
+        <mass value="${post_mass}"/>
+        <inertia
+          ixx="${(post_mass/12) * (3*post_radius*post_radius + post_length*post_length)}"
+          iyy="${(post_mass/12) * (3*post_radius*post_radius + post_length*post_length)}"
+          izz="${(post_mass/2) * (post_radius*post_radius)}"
+          ixy="0"
+          ixz="0"
+          iyz="0"/>
+      </inertial>
     </link>
-    <joint name="${name}_joint" type="fixed">
-      <origin xyz="${x} ${y} ${z}" rpy="${R} ${P} ${Y}" />
+    <!-- Sensor post arm -->
+    <link name="${name}_post_arm_link">
+      <visual name="${name}_post_arm_visual">
+        <origin xyz="-0.038 0 -0.003" rpy="${radians(-60)} 0 ${-pi/2}"/>
+        <geometry>
+          <mesh filename="package://vrx_gazebo/models/sensor_post/mesh/sensor_post_arm.dae"/>
+        </geometry>
+      </visual>
+      <collision name="${name}_post_arm_collision">
+        <origin xyz="0 0 0" rpy="${radians(-60)-pi/20} 0 ${-pi/2}"/>
+        <geometry>
+          <cylinder radius="0.008" length="0.065"/>
+        </geometry>
+      </collision>
+      <inertial>
+        <origin xyz="0 0 0" rpy="${radians(-60)-pi/20} 0 ${-pi/2}"/>
+        <mass value="0.1"/>
+        <inertia
+          ixx="0.00003680833"
+          iyy="0.00003680833"
+          izz="0.00000320000"
+          ixy="0"
+          ixz="0"
+          iyz="0"/>
+      </inertial>
+    </link>
+    <!-- Base to sensor post joint -->
+    <xacro:property name="post_z" value="${platform_z+post_length/2}"/>
+    <xacro:property name="post_to_lidar_x" value="${post_to_post_arm_x+post_arm_to_lidar_x}"/>
+    <joint name="base_to_${name}_post_joint" type="fixed">
+      <origin xyz="${x-(post_to_lidar_x)*cos(post_Y)} ${y-(post_to_lidar_x)*sin(post_Y)} ${post_z}" rpy="0 0 ${post_Y}" />
       <parent link="base_link" />
+      <child link="${name}_post_link" />
+    </joint>
+    <!-- Sensor post to sensor post arm joint -->
+    <joint name="${name}_post_to_${name}_post_arm_joint" type="fixed">
+      <origin xyz="${post_to_post_arm_x} 0 ${z-post_z-post_arm_to_lidar_z}" rpy="0 0 0" />
+      <parent link="${name}_post_link" />
+      <child link="${name}_post_arm_link" />
+    </joint>
+    <!-- Sensor post arm to lidar joint -->
+    <joint name="${name}_post_arm_to_${name}_joint" type="fixed">
+      <origin xyz="${post_arm_to_lidar_x} 0 ${post_arm_to_lidar_z}" rpy="${R} ${P} ${Y-post_Y}" />
+      <parent link="${name}_post_arm_link" />
       <child link="${name}_link" />
     </joint>
@@ -52,5 +154,5 @@
           </scan>
           <range>
-            <min>0.05</min>
+            <min>0.1</min>
             <max>${max_range}</max>
           </range>
@@ -64,7 +166,12 @@
           <topicName>${name}/points</topicName>
           <frameName>${name}_link</frameName>
+          <min_intensity>0</min_intensity>
         </plugin>
       </sensor>
     </gazebo>
+    <!-- Set color of post -->
+    <gazebo reference="${name}_post_link">
+      <material>Gazebo/Black</material>
+    </gazebo>
   </xacro:macro>
 </robot>
