Commit message: Imported upstream version '1.1.0' of 'upstream'

File: wamv_gazebo/urdf/sensors/wamv_camera.xacro (robot description, xacro)
@@ -1,28 +1,120 @@
 <?xml version="1.0"?>
 <robot xmlns:xacro="http://ros.org/wiki/xacro">
-  <xacro:macro name="wamv_camera" params="name x:=0.5 y:=0 z:=1.5 R:=0 P:=0 Y:=0">
+  <xacro:macro name="wamv_camera" params="name x:=0.5 y:=0 z:=1.5 R:=0 P:=0 Y:=0 post_Y:=0">
+    <!-- Define length variables for link positioning -->
+    <xacro:property name="platform_z" value="1.2965"/>
+    <xacro:property name="post_to_post_arm_x" value="0.03"/>
+    <xacro:property name="post_arm_to_camera_x" value="0.02"/>
+    <xacro:property name="post_arm_to_camera_z" value="0.027"/>
+    <!-- Monocular Camera -->
     <link name="${name}_link">
       <visual name="${name}_visual">
-        <xacro:property name="visual_length" value="0.05" />
-        <origin xyz="-${visual_length/2.0} 0 0" rpy="0 1.57 0" />
+        <origin xyz="-0.033 0 0" rpy="0 0 ${pi/2}"/>
         <geometry>
-          <cylinder radius="0.01" length="${visual_length}" />
+          <mesh filename="package://vrx_gazebo/models/mono_camera/mesh/mono_camera.dae"/>
         </geometry>
-        <material name="${name}_visual_material">
-          <color rgba="1.0 1.0 0.0 1.0" />
+      </visual>
+      <collision name="${name}_lens_collision">
+        <origin xyz="0.018 0 0" rpy="0 ${pi/2} 0"/>
+        <geometry>
+          <cylinder radius="0.015" length="0.042"/>
+        </geometry>
+      </collision>
+      <collision name="${name}_box_collision">
+        <origin xyz="-0.0205 0 0" rpy="0 0 0"/>
+        <geometry>
+          <box size="0.036 0.03 0.03"/>
+        </geometry>
+      </collision>
+      <!-- Model inertia as box with <size>0.078 0.03 0.03</size> -->
+      <inertial>
+        <mass value="0.3"/>
+        <inertia
+          ixx="0.0000450"
+          iyy="0.0001746"
+          izz="0.0001746"
+          ixy="0"
+          ixz="0"
+          iyz="0"/>
+      </inertial>
+    </link>
+    <!-- Define post length and mass based on desired z position of sensor -->
+    <xacro:property name="post_length" value="${z-platform_z-post_arm_to_camera_z}"/>
+    <xacro:property name="post_mass_per_meter" value="0.9"/>
+    <xacro:property name="post_mass" value="${post_mass_per_meter * post_length}"/>
+    <xacro:property name="post_radius" value="0.0076"/>
+    <!-- Sensor post -->
+    <link name="${name}_post_link">
+      <visual>
+        <geometry>
+          <cylinder radius="${post_radius}" length="${post_length}"/>
+        </geometry>
+        <material name="${name}_post_material">
+          <color rgba="0.0 0.0 0.0 1.0"/>
         </material>
       </visual>
+      <collision name="${name}_post_collision">
+        <geometry>
+          <cylinder radius="${post_radius}" length="${post_length}"/>
+        </geometry>
+      </collision>
+      <inertial>
+        <mass value="${post_mass}"/>
+        <inertia
+          ixx="${(post_mass/12) * (3*post_radius*post_radius + post_length*post_length)}"
+          iyy="${(post_mass/12) * (3*post_radius*post_radius + post_length*post_length)}"
+          izz="${(post_mass/2) * (post_radius*post_radius)}"
+          ixy="0"
+          ixz="0"
+          iyz="0"/>
+      </inertial>
     </link>
-    <joint name="${name}_joint" type="fixed">
-      <origin xyz="${x} ${y} ${z}" rpy="${R} ${P} ${Y}"/>
-      <parent link="base_link"/>
-      <child link="${name}_link"/>
+    <!-- Sensor post arm -->
+    <link name="${name}_post_arm_link">
+      <visual name="${name}_post_arm_visual">
+        <origin xyz="-0.038 0 -0.003" rpy="${radians(-60)} 0 ${-pi/2}"/>
+        <geometry>
+          <mesh filename="package://vrx_gazebo/models/sensor_post/mesh/sensor_post_arm.dae"/>
+        </geometry>
+      </visual>
+      <collision name="${name}_post_arm_collision">
+        <origin xyz="0 0 0" rpy="${radians(-60)-pi/20} 0 ${-pi/2}"/>
+        <geometry>
+          <cylinder radius="0.008" length="0.065"/>
+        </geometry>
+      </collision>
+      <inertial>
+        <origin xyz="0 0 0" rpy="${radians(-60)-pi/20} 0 ${-pi/2}"/>
+        <mass value="0.1"/>
+        <inertia
+          ixx="0.00003680833"
+          iyy="0.00003680833"
+          izz="0.00000320000"
+          ixy="0"
+          ixz="0"
+          iyz="0"/>
+      </inertial>
+    </link>
+    <!-- Base to sensor post joint -->
+    <xacro:property name="post_z" value="${platform_z+post_length/2}"/>
+    <xacro:property name="post_to_camera_x" value="${post_to_post_arm_x+post_arm_to_camera_x}"/>
+    <joint name="base_to_${name}_post_joint" type="fixed">
+      <origin xyz="${x-(post_to_camera_x)*cos(post_Y)} ${y-(post_to_camera_x)*sin(post_Y)} ${post_z}" rpy="0 0 ${post_Y}" />
+      <parent link="base_link" />
+      <child link="${name}_post_link" />
     </joint>
-    <link name="${name}_link_optical" />
-    <joint name="${name}_optical_joint" type="fixed">
-      <origin xyz="0 0 0" rpy="${-pi/2} 0 ${-pi/2}" />
-      <parent link="${name}_link"/>
-      <child link="${name}_link_optical"/>
+    <!-- Sensor post to sensor post arm joint -->
+    <joint name="${name}_post_to_${name}_post_arm_joint" type="fixed">
+      <origin xyz="${post_to_post_arm_x} 0 ${z-post_z-post_arm_to_camera_z}" rpy="0 0 0" />
+      <parent link="${name}_post_link" />
+      <child link="${name}_post_arm_link" />
     </joint>
+    <!-- Sensor post arm to camera joint -->
+    <joint name="${name}_post_arm_to_${name}_joint" type="fixed">
+      <origin xyz="${post_arm_to_camera_x} 0 ${post_arm_to_camera_z}" rpy="${R} ${P} ${Y-post_Y}" />
+      <parent link="${name}_post_arm_link" />
+      <child link="${name}_link" />
+    </joint>
+    <!-- Gazebo camera setup -->
     <gazebo reference="${name}_link">
       <sensor type="camera" name="${name}_sensor">
@@ -31,10 +123,10 @@
           <horizontal_fov>1.3962634</horizontal_fov>
           <image>
-            <width>800</width>
-            <height>800</height>
+            <width>1280</width>
+            <height>720</height>
             <format>R8G8B8</format>
           </image>
           <clip>
-            <near>0.02</near>
+            <near>0.05</near>
             <far>300</far>
           </clip>
@@ -64,4 +156,8 @@
       </sensor>
     </gazebo>
+    <!-- Set color of post -->
+    <gazebo reference="${name}_post_link">
+      <material>Gazebo/Black</material>
+    </gazebo>
   </xacro:macro>
 </robot>

File: wamv_gazebo/urdf/sensors/wamv_gps.xacro (robot description, xacro)
@@ -1,23 +1,27 @@
 <?xml version="1.0" encoding="UTF-8"?>
 <robot xmlns:xacro="http://ros.org/wiki/xacro">
-  <xacro:macro name="wamv_gps" params="name:=gps x:=0 y:=0 z:=1.3 R:=0 P:=0 Y:=0">
+  <xacro:macro name="wamv_gps" params="name:=gps x:=0.3 y:=0 z:=1.3 R:=0 P:=0 Y:=0">
     <link name="${name}_link">
-      <visual name="${name}_visual_base">
+      <visual name="${name}_visual">
         <geometry>
-          <box size="0.1 0.1 0.025" />
+          <mesh filename="package://wamv_gazebo/mesh/gps.dae"/>
         </geometry>
-        <material name="${name}_visual_base_material">
-          <color rgba="1.0 1.0 1.0 1.0" />
-        </material>
       </visual>
-      <visual name="${name}_visual_antenna">
-        <origin xyz="0 0 0.025" />
+      <collision name="${name}_collision_base">
+        <origin xyz="0 0 0.025" rpy="0 0 0" />
         <geometry>
-          <sphere radius="0.03" />
+          <cylinder length="0.05" radius="0.015" />
         </geometry>
-        <material name="${name}_visual_antenna_material">
-          <color rgba="0.7 0.7 0.7 1.0" />
-        </material>
-      </visual>
+      </collision>
+      <collision name="${name}_collision_antenna">
+        <origin xyz="0 0 0.11" rpy="0 0 0" />
+        <geometry>
+          <cylinder length="0.1" radius="0.15" />
+        </geometry>
+      </collision>
+      <inertial>
+        <mass value="1"/>
+        <inertia ixx="0.006458" ixy="0.0" ixz="0.0" iyy="0.006458" iyz="0.0" izz="0.01125"/>
+      </inertial>
     </link>
     <joint name="${name}_joint" type="fixed">
@@ -33,4 +37,9 @@
         <frameId>${name}_link</frameId>
         <topicName>gps/fix</topicName>
+        <!-- Note that the hector_gazebo_ros_gps plugin uses NWU coordinates
+             for reporting velocities.  This may cause problems if localization
+             requires velocity in ENU.
+             See Issue #64 in VRX project for details
+             https://bitbucket.org/osrf/vrx/issues/64 -->
         <velocityTopicName>gps/fix_velocity</velocityTopicName>
         <!-- Location of origin of Gazebo Sand Island map -->

File: wamv_gazebo/urdf/wamv_gazebo.urdf.xacro (robot description, xacro)
@@ -11,21 +11,38 @@
   <xacro:arg name="ground_truth_enabled" default="false" />
   <xacro:arg name="vrx_sensors_enabled" default="false" />
+  <!-- Sensor yaml file -->
+  <xacro:arg name="yaml_sensor_generation" default="false"/>
+  <xacro:arg name="sensor_xacro_file" default = ""/>
+  <!-- Thruster yaml file -->
+  <xacro:arg name="yaml_thruster_generation" default="false"/>
+  <xacro:arg name="thruster_xacro_file" default = ""/>
   <!-- === The WAM-V platform === -->
-  <xacro:include filename="$(find wamv_gazebo)/urdf/wamv_gazebo.xacro" />
+  <xacro:include filename="$(find wamv_gazebo)/urdf/wamv_gazebo.xacro"/>
+  <!-- === Batteries === -->
+  <xacro:include filename="$(find wamv_description)/urdf/battery.xacro"/>
+  <xacro:battery prefix="left" position="0 1 0.45" orientation="0 0 0"/>
+  <xacro:battery prefix="right" position="0 -1 0.45" orientation="0 0 0"/>
   <!-- === Thrusters === -->
-  <xacro:property name="thruster_conf" value="$(arg thruster_config)"/> -->
-  <!-- Default WAM-V with two aft thrusters -->
-  <xacro:if value="${thruster_conf == 'H'}">
-     <xacro:wamv_gazebo thruster_layout="$(find wamv_gazebo)/urdf/thruster_layouts/wamv_aft_thrusters.xacro"/>
+  <!-- Use thruster yaml file if given -->
+  <xacro:if value="$(arg yaml_thruster_generation)">
+    <xacro:wamv_gazebo thruster_layout="$(arg thruster_xacro_file)"/>
   </xacro:if>
-  <!-- WAMV with "T" thruster configuration -->
-  <xacro:if value="${thruster_conf == 'T'}">
-    <xacro:wamv_gazebo thruster_layout="$(find wamv_gazebo)/urdf/thruster_layouts/wamv_t_thrusters.xacro"/>
-  </xacro:if>
-  <!-- WAMV with "X" thruster configuration -->
-  <xacro:if value="${thruster_conf == 'X'}">
-    <xacro:wamv_gazebo thruster_layout="$(find wamv_gazebo)/urdf/thruster_layouts/wamv_x_thrusters.xacro"/>
-  </xacro:if>
-  <!-- Decide if we lock the robot to the world -->
+  <!-- Otherwise, add thrusters based on thruster_config variable -->
+  <xacro:unless value="$(arg yaml_thruster_generation)">
+    <xacro:property name="thruster_conf" value="$(arg thruster_config)"/>
+    <!-- Default WAM-V with two aft thrusters -->
+    <xacro:if value="${thruster_conf == 'H'}">
+       <xacro:wamv_gazebo thruster_layout="$(find wamv_gazebo)/urdf/thruster_layouts/wamv_aft_thrusters.xacro"/>
+    </xacro:if>
+    <!-- WAMV with "T" thruster configuration -->
+    <xacro:if value="${thruster_conf == 'T'}">
+      <xacro:wamv_gazebo thruster_layout="$(find wamv_gazebo)/urdf/thruster_layouts/wamv_t_thrusters.xacro"/>
+    </xacro:if>
+    <!-- WAMV with "X" thruster configuration -->
+    <xacro:if value="${thruster_conf == 'X'}">
+      <xacro:wamv_gazebo thruster_layout="$(find wamv_gazebo)/urdf/thruster_layouts/wamv_x_thrusters.xacro"/>
+    </xacro:if>
+  </xacro:unless>
+  <!-- === Decide if we lock the robot to the world === -->
   <xacro:if value="$(arg locked)">
     <gazebo>
@@ -54,37 +71,49 @@
     </gazebo>
   </xacro:if>
-  <!-- Add a front camera -->
-  <xacro:if value="$(arg camera_enabled)">
-    <xacro:wamv_camera name="front_camera" y="0.3" x="0.75" P="${radians(15)}" />
+  <!-- === Sensors === -->
+  <!-- Use sensor yaml file if given -->
+  <xacro:if value="$(arg yaml_sensor_generation)">
+    <xacro:include filename="$(arg sensor_xacro_file)"/>
+    <xacro:yaml_sensors />
   </xacro:if>
-  <!-- Add simulated GPS -->
-  <xacro:if value="$(arg gps_enabled)">
-    <xacro:wamv_gps name="gps_wamv" y="0.2" />
-  </xacro:if>
-  <!-- Add Simulated IMU -->
-  <xacro:if value="$(arg imu_enabled)">
-    <xacro:wamv_imu name="imu_wamv" y="-0.2" />
-  </xacro:if>
-  <!-- Add 3D LIDAR -->
-  <xacro:if value="$(arg lidar_enabled)">
-    <xacro:wamv_3d_lidar name="lidar_wamv" y="-0.3" />
-  </xacro:if>
-  <!-- Add P3D ground truth -->
-  <xacro:if value="$(arg ground_truth_enabled)">
-    <xacro:wamv_p3d name="p3d_wamv"/>
-  </xacro:if>
-  <!-- ==== VRX sensor configuration ==== -->
-  <xacro:if value="$(arg vrx_sensors_enabled)">
-    <!-- Add a stereo camera pair -->
-    <xacro:wamv_camera name="front_left_camera" y="0.1" x="0.75" P="${radians(15)}" />
-    <xacro:wamv_camera name="front_right_camera" y="-0.1" x="0.75" P="${radians(15)}" />
-    <!-- Add a camera facing right -->
-    <xacro:wamv_camera name="middle_right_camera" y="-0.45" P="${radians(15)}" Y="${radians(-90)}" />
+  <!-- Otherwise, add sensors based on enable variables -->
+  <xacro:unless value="$(arg yaml_sensor_generation)">
+    <!-- Add a front camera -->
+    <xacro:if value="$(arg camera_enabled)">
+      <xacro:wamv_camera name="front_camera" y="0.3" x="0.75" P="${radians(15)}" />
+    </xacro:if>
     <!-- Add simulated GPS -->
-    <xacro:wamv_gps name="gps_wamv" y="0.2" />
+    <xacro:if value="$(arg gps_enabled)">
+      <xacro:wamv_gps name="gps_wamv" x="-0.85" />
+    </xacro:if>
     <!-- Add Simulated IMU -->
-    <xacro:wamv_imu name="imu_wamv" y="-0.2" />
+    <xacro:if value="$(arg imu_enabled)">
+      <xacro:wamv_imu name="imu_wamv" y="-0.2" />
+    </xacro:if>
     <!-- Add 3D LIDAR -->
-    <xacro:wamv_3d_lidar name="lidar_wamv" P="${radians(8)}" />
-  </xacro:if>
+    <xacro:if value="$(arg lidar_enabled)">
+      <xacro:lidar name="lidar_wamv" y="-0.3" type="16_beam"/>
+    </xacro:if>
+    <!-- Add P3D ground truth -->
+    <xacro:if value="$(arg ground_truth_enabled)">
+      <xacro:wamv_p3d name="p3d_wamv"/>
+    </xacro:if>
+    <!-- ==== VRX sensor configuration ==== -->
+    <xacro:if value="$(arg vrx_sensors_enabled)">
+      <!-- Add CPU Cases -->
+      <xacro:include filename="$(find wamv_description)/urdf/cpu_cases.xacro" />
+      <xacro:cpu_cases position="-0.15 0 1.53" orientation="0 0 0"/>
+      <!-- Add a stereo camera pair -->
+      <xacro:wamv_camera name="front_left_camera" y="0.1" x="0.75" P="${radians(15)}" />
+      <xacro:wamv_camera name="front_right_camera" y="-0.1" x="0.75" P="${radians(15)}" />
+      <!-- Add a camera facing right -->
+      <xacro:wamv_camera name="middle_right_camera" y="-0.45" P="${radians(15)}" Y="${radians(-90)}" post_Y="${radians(-90)}" />
+      <!-- Add simulated GPS -->
+      <xacro:wamv_gps name="gps_wamv" x="-0.85" />
+      <!-- Add Simulated IMU -->
+      <xacro:wamv_imu name="imu_wamv" y="-0.2" />
+      <!-- Add 3D LIDAR -->
+      <xacro:lidar name="lidar_wamv" type="16_beam"/>
+    </xacro:if>
+  </xacro:unless>
 </robot>
