Commit message: Rebase from 'upstream'

File: vrx_gazebo/worlds/dock.world.xacro (robot description, xacro)
@@ -8,39 +8,20 @@
     <xacro:include filename="$(find wave_gazebo)/world_models/ocean_waves/model.xacro"/>
     <xacro:ocean_waves/>
+    <!--wind for the wamv-->
+    <xacro:include filename="$(find vrx_gazebo)/worlds/xacros/usv_wind_plugin.xacro"/>
+    <xacro:usv_wind_gazebo>
+      <wind_objs>
+        <wind_obj>
+          <name>wamv</name>
+          <link_name>base_link</link_name>
+          <coeff_vector>.5 .5 .33</coeff_vector>
+        </wind_obj>
+      </wind_objs>
+    </xacro:usv_wind_gazebo>
     <!-- The 2018 dock with the two placards -->
     <include>
-      <uri>model://dock_2018</uri>
-      <pose>60 -2.75 0 0 0 0</pose>
+      <uri>model://dock_2018_dynamic</uri>
+      <pose>130 97 0 0 0 0</pose>
     </include>
-    <!-- Uncomment to visualize the bay #1 activation zone -->
-    <!-- <model name="activation_placard1">
-      <static>true</static>
-      <link name="link">
-        <visual name="visual">
-          <pose>72.75 0 0 0 0 0</pose>
-          <geometry>
-            <box>
-              <size>1.5 4 2</size>
-            </box>
-          </geometry>
-          <transparency>0.8</transparency>
-        </visual>
-      </link>
-    </model> -->
-    <!-- Uncomment to visualize the bay #2 activation zone -->
-    <!-- <model name="activation_placard2">
-      <static>true</static>
-      <link name="link">
-        <visual name="visual">
-          <pose>61.75 0 0 0 0 0</pose>
-          <geometry>
-            <box>
-              <size>1.5 4 2</size>
-            </box>
-          </geometry>
-          <transparency>0.8</transparency>
-        </visual>
-      </link>
-    </model> -->
     <!-- The scoring plugin -->
     <plugin name="scan_dock_scoring_plugin"
@@ -70,5 +51,6 @@
         <bay>
           <name>bay1</name>
-          <activation_topic>/vrx/dock_2018/bay_1/contain</activation_topic>
+          <internal_activation_topic>/vrx/dock_2018/bay_1_internal/contain</internal_activation_topic>
+          <external_activation_topic>/vrx/dock_2018/bay_1_external/contain</external_activation_topic>
           <symbol_topic>/vrx/dock_2018_placard1/symbol</symbol_topic>
           <min_dock_time>10.0</min_dock_time>
@@ -78,5 +60,6 @@
         <bay>
           <name>bay2</name>
-          <activation_topic>/vrx/dock_2018/bay_2/contain</activation_topic>
+          <internal_activation_topic>/vrx/dock_2018/bay_2_internal/contain</internal_activation_topic>
+          <external_activation_topic>/vrx/dock_2018/bay_2_external/contain</external_activation_topic>
           <symbol_topic>/vrx/dock_2018_placard2/symbol</symbol_topic>
           <min_dock_time>10.0</min_dock_time>
@@ -91,5 +74,5 @@
     <plugin name="vehicle_docked_bay1" filename="libContainPlugin.so">
       <entity>wamv::base_link</entity>
-      <namespace>vrx/dock_2018/bay_1</namespace>
+      <namespace>vrx/dock_2018/bay_1_internal</namespace>
       <pose frame="robotx_dock_2018::dock_2018_placard1::placard::link">0 -5 -1.5 0 0 0</pose>
       <geometry>
@@ -99,8 +82,19 @@
       </geometry>
     </plugin>
+    <!-- Triggers a message when the vehicle enters and exits the bay #1 -->
+    <plugin name="vehicle_docked_bay1_exterior" filename="libContainPlugin.so">
+      <entity>wamv::base_link</entity>
+      <namespace>vrx/dock_2018/bay_1_external</namespace>
+      <pose frame="robotx_dock_2018::dock_2018_placard1::placard::link">0 -10 -1.5 0 0 0</pose>
+      <geometry>
+        <box>
+          <size>8 1.5 2</size>
+        </box>
+      </geometry>
+    </plugin>
     <!-- Triggers a message when the vehicle enters and exits the bay #2 -->
     <plugin name="vehicle_docked_bay2" filename="libContainPlugin.so">
       <entity>wamv::base_link</entity>
-      <namespace>vrx/dock_2018/bay_2</namespace>
+      <namespace>vrx/dock_2018/bay_2_internal</namespace>
       <pose frame="robotx_dock_2018::dock_2018_placard2::placard::link">0 5 -1.5 0 0 0</pose>
       <geometry>
@@ -110,4 +104,15 @@
       </geometry>
     </plugin>
+    <!-- Triggers a message when the vehicle enters and exits the bay #1 -->
+    <plugin name="vehicle_docked_bay2_exterior" filename="libContainPlugin.so">
+      <entity>wamv::base_link</entity>
+      <namespace>vrx/dock_2018/bay_2_external</namespace>
+      <pose frame="robotx_dock_2018::dock_2018_placard1::placard::link">0 10 -1.5 0 0 0</pose>
+      <geometry>
+        <box>
+          <size>8 1.5 2</size>
+        </box>
+      </geometry>
+    </plugin>
   </world>
 </sdf>

File: vrx_gazebo/worlds/scan_and_dock.world.xacro (robot description, xacro)
@@ -8,4 +8,15 @@
     <xacro:include filename="$(find wave_gazebo)/world_models/ocean_waves/model.xacro"/>
     <xacro:ocean_waves/>
+    <!--wind for the wamv-->
+    <xacro:include filename="$(find vrx_gazebo)/worlds/xacros/usv_wind_plugin.xacro"/>
+    <xacro:usv_wind_gazebo>
+      <wind_objs>
+        <wind_obj>
+          <name>wamv</name>
+          <link_name>base_link</link_name>
+          <coeff_vector>.5 .5 .33</coeff_vector>
+        </wind_obj>
+      </wind_objs>
+    </xacro:usv_wind_gazebo>
     <!-- The light buoy -->
     <include>
@@ -75,5 +86,6 @@
         <bay>
           <name>bay1</name>
-          <activation_topic>/vrx/dock_2018/bay_1/contain</activation_topic>
+          <internal_activation_topic>/vrx/dock_2018/bay_1/contain</internal_activation_topic>
+          <external_activation_topic>/vrx/dock_2018/bay_1_exterior/contain</external_activation_topic>
           <symbol_topic>/vrx/dock_2018_placard1/symbol</symbol_topic>
 	        <min_dock_time>10.0</min_dock_time>
@@ -83,5 +95,6 @@
         <bay>
           <name>bay2</name>
-          <activation_topic>/vrx/dock_2018/bay_2/contain</activation_topic>
+          <internal_activation_topic>/vrx/dock_2018/bay_2/contain</internal_activation_topic>
+          <external_activation_topic>/vrx/dock_2018/bay_2_exterior/contain</external_activation_topic>
           <symbol_topic>/vrx/dock_2018_placard2/symbol</symbol_topic>
           <min_dock_time>10.0</min_dock_time>

File: vrx_gazebo/worlds/xacros/dock.xacro (robot description, xacro)
@@ -2,5 +2,12 @@
 <!-- World containing sandisland model and some course challenges -->
 <world xmlns:xacro="http://ros.org/wiki/xacro">
-  <xacro:macro name="dock" params="uri:=dock_2018 x:=60 y:=-2.75 z:=0 R:=0 P:=0 Y:=0 bay1_allowed:=false bay1_symbol:=red_circle bay2_allowed:=true bay2_symbol:=blue_cross">
+  <xacro:macro name="dock" params="model_name:=robotx_dock_2018
+    uri:=dock_2018 x:=60 y:=-2.75 z:=0
+    R:=0 P:=0 Y:=0 bay1_allowed:=false bay1_symbol:=red_circle
+    bay2_allowed:=true bay2_symbol:=blue_cross
+    light_buoy_present:=false
+    color_1:=red color_2:=green color_3:=blue
+    lb_x:=90 lb_y:=70 lb_z:=0 lb_R:=0 lb_P:=0 lb_Y:=0
+    enable_color_checker:=true">
     <!-- The 2018 dock with the two placards -->
     <include>
@@ -8,4 +15,11 @@
       <pose>${x} ${y} ${z} ${R} ${P} ${Y}</pose>
     </include>
+    <!-- Add a ligth buoy if doing Scan and Dock -->
+    <xacro:if value="${light_buoy_present}">
+      <include>
+        <uri>model://robotx_light_buoy</uri>
+        <pose>${lb_x} ${lb_y} ${lb_z} ${lb_R} ${lb_P} ${lb_Y}</pose>
+      </include>
+    </xacro:if>
     <!-- The scoring plugin -->
     <plugin name="scan_dock_scoring_plugin"
@@ -26,14 +40,16 @@
       </release_joints>
       <!-- Color sequence checker -->
+      <enable_color_checker>${enable_color_checker}</enable_color_checker>
       <robot_namespace>vrx</robot_namespace>
       <color_sequence_service>scan_dock/color_sequence</color_sequence_service>
-      <color_1>red</color_1>
-      <color_2>green</color_2>
-      <color_3>blue</color_3>
+      <color_1>${color_1}</color_1>
+      <color_2>${color_2}</color_2>
+      <color_3>${color_3}</color_3>
       <!-- Dock checkers -->
       <bays>
         <bay>
           <name>bay1</name>
-          <activation_topic>/vrx/dock_2018/bay_1/contain</activation_topic>
+          <internal_activation_topic>/vrx/dock_2018/bay_1_internal/contain</internal_activation_topic>
+          <external_activation_topic>/vrx/dock_2018/bay_1_external/contain</external_activation_topic>
           <symbol_topic>/vrx/dock_2018_placard1/symbol</symbol_topic>
           <min_dock_time>10.0</min_dock_time>
@@ -43,5 +59,6 @@
         <bay>
           <name>bay2</name>
-          <activation_topic>/vrx/dock_2018/bay_2/contain</activation_topic>
+          <internal_activation_topic>/vrx/dock_2018/bay_2_internal/contain</internal_activation_topic>
+          <external_activation_topic>/vrx/dock_2018/bay_2_external/contain</external_activation_topic>
           <symbol_topic>/vrx/dock_2018_placard2/symbol</symbol_topic>
           <min_dock_time>10.0</min_dock_time>
@@ -54,6 +71,6 @@
     <plugin name="vehicle_docked_bay1" filename="libContainPlugin.so">
       <entity>wamv::base_link</entity>
-      <namespace>vrx/dock_2018/bay_1</namespace>
-      <pose frame="robotx_dock_2018::dock_2018_placard1::placard::link">0 -5 -1.5 0 0 0</pose>
+      <namespace>vrx/dock_2018/bay_1_internal</namespace>
+      <pose frame="${model_name}::dock_2018_placard1::placard::link">0 -5 -1.5 0 0 0</pose>
       <geometry>
         <box>
@@ -62,9 +79,20 @@
       </geometry>
     </plugin>
+    <!-- Triggers a message when the vehicle enters and exits the bay #1 -->
+    <plugin name="vehicle_docked_bay1_exterior" filename="libContainPlugin.so">
+      <entity>wamv::base_link</entity>
+      <namespace>vrx/dock_2018/bay_1_external</namespace>
+      <pose frame="${model_name}::dock_2018_placard1::placard::link">0 -10 -1.5 0 0 0</pose>
+      <geometry>
+        <box>
+          <size>8 1.5 2</size>
+        </box>
+      </geometry>
+    </plugin>
     <!-- Triggers a message when the vehicle enters and exits the bay #2 -->
     <plugin name="vehicle_docked_bay2" filename="libContainPlugin.so">
       <entity>wamv::base_link</entity>
-      <namespace>vrx/dock_2018/bay_2</namespace>
-      <pose frame="robotx_dock_2018::dock_2018_placard2::placard::link">0 5 -1.5 0 0 0</pose>
+      <namespace>vrx/dock_2018/bay_2_internal</namespace>
+      <pose frame="${model_name}::dock_2018_placard2::placard::link">0 5 -1.5 0 0 0</pose>
       <geometry>
         <box>
@@ -73,4 +101,15 @@
       </geometry>
     </plugin>
+    <!-- Triggers a message when the vehicle enters and exits the bay #1 -->
+    <plugin name="vehicle_docked_bay2_exterior" filename="libContainPlugin.so">
+      <entity>wamv::base_link</entity>
+      <namespace>vrx/dock_2018/bay_2_external</namespace>
+      <pose frame="${model_name}::dock_2018_placard1::placard::link">0 10 -1.5 0 0 0</pose>
+      <geometry>
+        <box>
+          <size>8 1.5 2</size>
+        </box>
+      </geometry>
+    </plugin>
   </xacro:macro>
 </world>
