Commit message: Rebase from 'release/kinetic/vrx_gazebo'

File: worlds/xacros/include_all_xacros.xacro (robot description, xacro)
@@ -1,7 +1,8 @@
 <?xml version="1.0"?>
 <world xmlns:xacro="http://ros.org/wiki/xacro">
-    <xacro:macro name="include_all_xacros">
+  <xacro:macro name="include_all_xacros">
     <xacro:include filename="$(find vrx_gazebo)/worlds/sandisland.xacro" />
-    <xacro:include filename="$(find vrx_gazebo)/worlds/xacros/sandisland2.xacro" />
+    <xacro:include filename="$(find vrx_gazebo)/worlds/xacros/sandisland_minus_scene.xacro" />
+    <xacro:include filename="$(find vrx_gazebo)/worlds/xacros/scene.xacro" />
     <xacro:include filename="$(find vrx_gazebo)/worlds/xacros/nav_challenge.xacro" />
     <xacro:include filename="$(find vrx_gazebo)/worlds/xacros/light_buoy.xacro" />
@@ -11,4 +12,10 @@
     <xacro:include filename="$(find vrx_gazebo)/worlds/xacros/scene_macro.xacro" />
     <xacro:include filename="$(find vrx_gazebo)/worlds/xacros/usv_wind_plugin.xacro" />
+    <xacro:include filename="$(find wave_gazebo)/world_models/ocean_waves/model.xacro"/>
+    <xacro:include filename="$(find vrx_gazebo)/worlds/xacros/perception.xacro" />
+    <xacro:include filename="$(find vrx_gazebo)/worlds/xacros/stationkeeping.xacro" />
+    <xacro:include filename="$(find vrx_gazebo)/worlds/xacros/dock.xacro" />
+    <xacro:include filename="$(find vrx_gazebo)/worlds/xacros/scan_and_dock.xacro" />
+    <xacro:include filename="$(find vrx_gazebo)/worlds/xacros/wayfinding.xacro" />
   </xacro:macro>
 </world>
